File: snowflake-v2.brd (EAGLE design)
At the start: 68.6 x 68.6 mm, 32 parts, among them J1 M03X2-NOSILK, J2 CON_TERMINAL_HOLES, U2 V_REG_MCP170X-CB

Commit message: Fixes.
Parts:
- moved R1 0.97 mm to (34.6, 24.1), turned to 244.6 degrees
- moved D12 0.64 mm to (39.9, 20.2)
- moved D19 0.64 mm to (39.9, 20.2)
Routing:
- net N$9: track 136.0 -> 155.6 mm, vias 6 -> 5
- net N$8: track 141.9 -> 151.0 mm
- net MOSI: track 22.5 -> 23.5 mm
- net N$7: track 146.5 -> 147.1 mm
