File: star.brd (EAGLE design)
At the start: 68.6 x 68.6 mm, 32 parts, among them J1 M03X2-NOSILK, J2 CON_TERMINAL_HOLES, U2 V_REG_MCP170X-CB

Commit message: It's a star, not a snowflake.
Parts:
- U2: value V_REG_MCP170X-CB -> V_REG_MCP170X-CB-NOSILK; device adi-misc:SOT23 -> snowflake:SOT23_NOSILK
- moved C2 1.88 mm to (39.0, 45.0), turned to 157.2 degrees
Connections:
- net GND: now also J2.P$5, J2.P$6; no longer J2.P$3, J2.P$4
- net N$1: now also J2.P$3, J2.P$4; no longer J2.P$5, J2.P$6
Routing:
- net N$1: track 11.5 -> 18.8 mm
- net GND: vias 14 -> 15
Changed lines of the file:
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@@
 <attribute name="VALUE" x="33.297221875" y="22.188378125" size="0.762" layer="27" font="vector" ratio="18" rot="R157.3"/>
 </element>
-<element name="C2" library="snowflake" package="C0805NOSILK" value="" x="39.751" y="46.736" smashed="yes" rot="R337.2">
-<attribute name="NAME" x="38.65665" y="48.229253125" size="0.762" layer="51" font="vector" ratio="18" rot="R337.2"/>
-<attribute name="VALUE" x="37.795396875" y="46.1804125" size="0.4064" layer="27" ratio="10" rot="R337.2"/>
+<element name="C2" library="snowflake" package="C0805NOSILK" value="" x="38.989" y="45.0215" smashed="yes" rot="R157.2">
+<attribute name="NAME" x="40.08335" y="43.528246875" size="0.762" layer="51" font="vector" ratio="18" rot="R157.2"/>
+<attribute name="VALUE" x="40.944603125" y="45.5770875" size="0.4064" layer="27" ratio="10" rot="R157.2"/>
 </element>
 <element name="C3" library="snowflake" package="C0805NOSILK" value="" x="44.831" y="43.688" smashed="yes" rot="R325.3">
@@
 <attribute name="VALUE" x="42.802859375" y="43.54760625" size="0.4064" layer="27" ratio="10" rot="R325.3"/>
 </element>
-<element name="U2" library="adi-misc" package="SOT23" value="V_REG_MCP170X-CB" x="48.133" y="46.228" smashed="yes" rot="R312.7">
+<element name="U2" library="snowflake" package="SOT23_NOSILK" value="V_REG_MCP170X-CB-NOSILK" x="48.133" y="46.228" smashed="yes" rot="R312.7">
 <attribute name="NAME" x="49.927603125" y="46.15591875" size="0.762" layer="51" font="vector" ratio="18" rot="R312.7"/>
 <attribute name="VALUE" x="44.50775" y="45.474853125" size="0.762" layer="27" ratio="10" rot="R312.7"/>
@@
 <contactref element="C3" pad="1"/>
 <contactref element="U2" pad="1"/>
-<contactref element="J2" pad="P$3"/>
-<contactref element="J2" pad="P$4"/>
 <wire x1="46.680340625" y1="46.180190625" x2="45.974" y2="46.228" width="0.4064" layer="1"/>
 <wire x1="45.974" y1="46.228" x2="43.9957" y2="44.2663875" width="0.4064" layer="1" curve="97.259662"/>
@@
 <via x="48.4505" y="27.8765" extent="1-16" drill="0.349759375"/>
 <via x="38.227" y="17.3355" extent="1-16" drill="0.349759375"/>
+<contactref element="J2" pad="P$6"/>
+<contactref element="J2" pad="P$5"/>
+<via x="37.211" y="43.053" extent="1-16" drill="0.349759375"/>
 </signal>
 <signal name="N$4">
@@
 <contactref element="C2" pad="2"/>
 <contactref element="U2" pad="3"/>
-<contactref element="J2" pad="P$5"/>
-<contactref element="J2" pad="P$6"/>
-<wire x1="40.6876125" y1="46.34228125" x2="41.021" y2="46.99" width="0.4064" layer="1"/>
-<wire x1="41.021" y1="46.99" x2="42.7433875" y2="47.62894375" width="0.4064" layer="1" curve="-84.823202"/>
 <wire x1="48.941403125" y1="46.973975" x2="48.387" y2="47.498" width="0.4064" layer="1"/>
-<wire x1="48.387" y1="47.498" x2="45.085" y2="47.371" width="0.4064" layer="1" curve="91.178102"/>
-<wire x1="45.085" y1="47.371" x2="42.7433875" y2="47.62894375" width="0.4064" layer="1" curve="-108.155682"/>
-<wire x1="42.7433875" y1="47.62894375" x2="43.727675" y2="49.970475" width="0.4064" layer="1"/>
+<contactref element="J2" pad="P$3"/>
+<contactref element="J2" pad="P$4"/>
+<wire x1="48.387" y1="47.498" x2="45.1485" y2="47.498" width="0.4064" layer="1" curve="86.772949"/>
+<wire x1="45.1485" y1="47.498" x2="43.4975" y2="46.101" width="0.4064" layer="1" curve="-6.300233"/>
+<wire x1="43.4975" y1="46.101" x2="41.0845" y2="46.0375" width="0.4064" layer="1" curve="-71.157663"/>
+<wire x1="41.0845" y1="46.0375" x2="39.5605" y2="46.5455" width="0.4064" layer="1" curve="31.272886"/>
+<wire x1="39.5605" y1="46.5455" x2="38.052384375" y2="45.415215625" width="0.4064" layer="1" curve="79.297144"/>
+<wire x1="39.044609375" y1="51.939053125" x2="38.060321875" y2="49.597521875" width="0.4064" layer="1"/>
+<wire x1="38.060321875" y1="49.597521875" x2="38.227" y2="48.0695" width="0.4064" layer="1" curve="58.050332"/>
+<wire x1="38.227" y1="48.0695" x2="38.052384375" y2="45.415215625" width="0.4064" layer="1" curve="-78.02848"/>
 </signal>
 </signals>

Commit message: Removed redundant cap.
Parts:
- removed C3: (no value), snowflake:C0805NOSILK
- J1: value M03X2-NOSILK -> CON_TERMINAL_HOLES; device snowflake:2X03_LOCK_NOSILK -> adi-misc:TERMINAL_2P_4H
- J2: value CON_TERMINAL_HOLES -> M03X2-NOSILK; device adi-misc:TERMINAL_2P_4H -> snowflake:2X03_LOCK_NOSILK
- U1: value (none) -> V_REG_MCP170X-CB-NOSILK; device snowflake:SOP8-8S2-NOSILK -> snowflake:SOT23_NOSILK
- U2: value V_REG_MCP170X-CB-NOSILK -> (none); device snowflake:SOT23_NOSILK -> snowflake:SOP8-8S2-NOSILK
- moved J1 32.8 mm to (40.9, 49.8), turned to 337.2 degrees
- moved J2 32.8 mm to (28.1, 19.6), turned to 157.3 degrees
- moved U1 18.3 mm to (48.1, 46.2), turned to 312.7 degrees
- moved U2 18.3 mm to (34.3, 34.3), turned to 270 degrees
- moved C1 7.72 mm to (39.0, 45.0), turned to 157.2 degrees
- moved C2 5.99 mm to (44.8, 43.7), turned to 325.3 degrees
- moved R1 0.79 mm to (34.8, 23.4), turned to 317.5 degrees
Connections:
- net GND: now also J1.P$5, J1.P$6, J2.6, U1.1, U2.4; no longer C3.1, J1.6, J2.P$5, J2.P$6, U1.4, U2.1
- net MISO: now also J2.1, U2.6; no longer J1.1, U1.6
- net MOSI: now also J2.4, U2.5; no longer J1.4, U1.5
- net N$1: now also C1.2, J1.P$3, J1.P$4, U1.3; no longer C2.2, J2.P$3, J2.P$4, U2.3
- net N$4: now also U2.2; no longer U1.2
- net N$5: now also U2.3; no longer U1.3
- net RST: now also J2.5, U2.1; no longer J1.5, U1.1
- net SCK: now also J2.3, U2.7; no longer J1.3, U1.7
- net VCC: now also C2.2, J2.2, U1.2, U2.8; no longer C1.2, C3.2, J1.2, U1.8, U2.2
Routing:
- net VCC: track 43.1 -> 39.3 mm
- net MOSI: track 23.5 -> 22.2 mm
- net N$9: track 155.6 -> 154.9 mm
Other:
- board text added: "Adi Linden"
- board text added: "Designed by"

Commit message: Created png. Added values to schematic.
Parts:
- C1: value (none) -> 1u
- C2: value (none) -> 10u
- R1, R2, R3, R4, R5: value (none) -> 47
- U1: value V_REG_MCP170X-CB-NOSILK -> MCP1702-5V
Changed lines of the file:
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@@
 </autorouter>
 <elements>
-<element name="R1" library="snowflake" package="R0805NOSILK" value="" x="34.798" y="23.368" smashed="yes" rot="R317.5">
+<element name="R1" library="snowflake" package="R0805NOSILK" value="47" x="34.798" y="23.368" smashed="yes" rot="R317.5">
 <attribute name="NAME" x="34.271071875" y="25.142753125" size="0.762" layer="51" font="vector" ratio="18" rot="R317.5"/>
 <attribute name="VALUE" x="32.769571875" y="23.50415" size="0.4064" layer="27" ratio="10" rot="R317.5"/>
 </element>
-<element name="R2" library="snowflake" package="R0805NOSILK" value="" x="43.18" y="29.21" smashed="yes">
+<element name="R2" library="snowflake" package="R0805NOSILK" value="47" x="43.18" y="29.21" smashed="yes">
 <attribute name="NAME" x="41.5925" y="30.1625" size="0.762" layer="51" font="vector" ratio="18"/>
 <attribute name="VALUE" x="41.5925" y="27.94" size="0.4064" layer="27" ratio="10"/>
 </element>
-<element name="R3" library="snowflake" package="R0805NOSILK" value="" x="43.18" y="39.37" smashed="yes">
+<element name="R3" library="snowflake" package="R0805NOSILK" value="47" x="43.18" y="39.37" smashed="yes">
 <attribute name="NAME" x="41.5925" y="40.3225" size="0.762" layer="51" font="vector" ratio="18"/>
 <attribute name="VALUE" x="41.5925" y="38.1" size="0.4064" layer="27" ratio="10"/>
 </element>
-<element name="R4" library="snowflake" package="R0805NOSILK" value="" x="25.4" y="39.37" smashed="yes" rot="R180">
+<element name="R4" library="snowflake" package="R0805NOSILK" value="47" x="25.4" y="39.37" smashed="yes" rot="R180">
 <attribute name="NAME" x="26.9875" y="38.4175" size="0.762" layer="51" font="vector" ratio="18" rot="R180"/>
 <attribute name="VALUE" x="26.9875" y="40.64" size="0.4064" layer="27" ratio="10" rot="R180"/>
 </element>
-<element name="R5" library="snowflake" package="R0805NOSILK" value="" x="25.4" y="29.21" smashed="yes" rot="R180">
+<element name="R5" library="snowflake" package="R0805NOSILK" value="47" x="25.4" y="29.21" smashed="yes" rot="R180">
 <attribute name="NAME" x="26.9875" y="28.2575" size="0.762" layer="51" font="vector" ratio="18" rot="R180"/>
 <attribute name="VALUE" x="26.9875" y="30.48" size="0.4064" layer="27" ratio="10" rot="R180"/>
@@
 <attribute name="VALUE" x="33.297221875" y="22.188378125" size="0.762" layer="27" font="vector" ratio="18" rot="R157.3"/>
 </element>
-<element name="C1" library="snowflake" package="C0805NOSILK" value="" x="38.989" y="45.0215" smashed="yes" rot="R157.2">
+<element name="C1" library="snowflake" package="C0805NOSILK" value="1u" x="38.989" y="45.0215" smashed="yes" rot="R157.2">
 <attribute name="NAME" x="40.08335" y="43.528246875" size="0.762" layer="51" font="vector" ratio="18" rot="R157.2"/>
 <attribute name="VALUE" x="40.944603125" y="45.5770875" size="0.4064" layer="27" ratio="10" rot="R157.2"/>
 </element>
-<element name="C2" library="snowflake" package="C0805NOSILK" value="" x="44.831" y="43.688" smashed="yes" rot="R325.3">
+<element name="C2" library="snowflake" package="C0805NOSILK" value="10u" x="44.831" y="43.688" smashed="yes" rot="R325.3">
 <attribute name="NAME" x="44.068084375" y="45.374821875" size="0.762" layer="51" font="vector" ratio="18" rot="R325.3"/>
 <attribute name="VALUE" x="42.802859375" y="43.54760625" size="0.4064" layer="27" ratio="10" rot="R325.3"/>
 </element>
-<element name="U1" library="snowflake" package="SOT23_NOSILK" value="V_REG_MCP170X-CB-NOSILK" x="48.133" y="46.228" smashed="yes" rot="R312.7">
+<element name="U1" library="snowflake" package="SOT23_NOSILK" value="MCP1702-5V" x="48.133" y="46.228" smashed="yes" rot="R312.7">
 <attribute name="NAME" x="49.927603125" y="46.15591875" size="0.762" layer="51" font="vector" ratio="18" rot="R312.7"/>
 <attribute name="VALUE" x="44.50775" y="45.474853125" size="0.762" layer="27" ratio="10" rot="R312.7"/>
