File: tree.brd (EAGLE design)
At the start: 62.9 x 69.8 mm, 31 parts, among them J1 M03X2-NOSILK, J2 CON_TERMINAL_HOLES, U2 MCP1702-5

Commit message: Created png. Added values to schematic.
Parts:
- C2: value (none) -> 1u
- C3: value (none) -> 10u
- R1, R2, R3, R4, R5: value (none) -> 47
- U2: value MCP1702-5 -> MCP1702-5V
Changed lines of the file:
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@@
 </autorouter>
 <elements>
-<element name="C2" library="snowflake" package="C0805NOSILK" value="" x="31.75" y="40.64" smashed="yes">
+<element name="C2" library="snowflake" package="C0805NOSILK" value="1u" x="31.75" y="40.64" smashed="yes">
 <attribute name="NAME" x="30.1625" y="41.5925" size="0.762" layer="51" font="vector" ratio="18"/>
 <attribute name="VALUE" x="30.1625" y="39.37" size="0.4064" layer="27" ratio="10"/>
 </element>
-<element name="C3" library="snowflake" package="C0805NOSILK" value="" x="31.75" y="31.75" smashed="yes">
+<element name="C3" library="snowflake" package="C0805NOSILK" value="10u" x="31.75" y="31.75" smashed="yes">
 <attribute name="NAME" x="30.1625" y="32.7025" size="0.762" layer="51" font="vector" ratio="18"/>
 <attribute name="VALUE" x="30.1625" y="30.48" size="0.4064" layer="27" ratio="10"/>
@@
 </element>
 <element name="J2" library="adi-misc" package="TERMINAL_2P_4H" value="CON_TERMINAL_HOLES" x="31.75" y="48.895" smashed="yes" rot="R90"/>
-<element name="R1" library="snowflake" package="R0805NOSILK" value="" x="39.37" y="21.59" smashed="yes">
+<element name="R1" library="snowflake" package="R0805NOSILK" value="47" x="39.37" y="21.59" smashed="yes">
 <attribute name="NAME" x="37.7825" y="22.5425" size="0.762" layer="51" font="vector" ratio="18"/>
 <attribute name="VALUE" x="37.7825" y="20.32" size="0.4064" layer="27" ratio="10"/>
 </element>
-<element name="R2" library="snowflake" package="R0805NOSILK" value="" x="39.37" y="24.13" smashed="yes">
+<element name="R2" library="snowflake" package="R0805NOSILK" value="47" x="39.37" y="24.13" smashed="yes">
 <attribute name="NAME" x="37.7825" y="25.0825" size="0.762" layer="51" font="vector" ratio="18"/>
 <attribute name="VALUE" x="37.7825" y="22.86" size="0.4064" layer="27" ratio="10"/>
 </element>
-<element name="R3" library="snowflake" package="R0805NOSILK" value="" x="39.37" y="30.48" smashed="yes">
+<element name="R3" library="snowflake" package="R0805NOSILK" value="47" x="39.37" y="30.48" smashed="yes">
 <attribute name="NAME" x="37.7825" y="31.4325" size="0.762" layer="51" font="vector" ratio="18"/>
 <attribute name="VALUE" x="37.7825" y="29.21" size="0.4064" layer="27" ratio="10"/>
 </element>
-<element name="R4" library="snowflake" package="R0805NOSILK" value="" x="24.13" y="30.48" smashed="yes" rot="R180">
+<element name="R4" library="snowflake" package="R0805NOSILK" value="47" x="24.13" y="30.48" smashed="yes" rot="R180">
 <attribute name="NAME" x="25.7175" y="29.5275" size="0.762" layer="51" font="vector" ratio="18" rot="R180"/>
 <attribute name="VALUE" x="25.7175" y="31.75" size="0.4064" layer="27" ratio="10" rot="R180"/>
 </element>
-<element name="R5" library="snowflake" package="R0805NOSILK" value="" x="24.13" y="24.13" smashed="yes" rot="R180">
+<element name="R5" library="snowflake" package="R0805NOSILK" value="47" x="24.13" y="24.13" smashed="yes" rot="R180">
 <attribute name="NAME" x="25.7175" y="23.1775" size="0.762" layer="51" font="vector" ratio="18" rot="R180"/>
 <attribute name="VALUE" x="25.7175" y="25.4" size="0.4064" layer="27" ratio="10" rot="R180"/>
@@
 <attribute name="VALUE" x="29.083" y="23.241" size="0.762" layer="27" font="vector" ratio="18"/>
 </element>
-<element name="U2" library="snowflake" package="SOT23_NOSILK" value="MCP1702-5" x="31.75" y="35.56" smashed="yes">
+<element name="U2" library="snowflake" package="SOT23_NOSILK" value="MCP1702-5V" x="31.75" y="35.56" smashed="yes">
 <attribute name="NAME" x="33.02" y="36.83" size="0.762" layer="51" font="vector" ratio="18"/>
 <attribute name="VALUE" x="29.845" y="32.385" size="0.762" layer="27" ratio="10"/>
